File: Diagostics Card.kicad_pcb (KiCad board)
At the start: 2 copper layers, 100 x 100 mm, 59 parts, among them J1 Conn_02x20_Odd_Even, SW1 SW_DIP_x01, SW2 Run, U1 74LS00, U2 74LS534, U3 GAL22V10B, U4 74LS14

Commit message: Corrected footprint and traces on Run button
Parts:
- SW2: footprint Button_Switch_THT:SW_TH_Tactile_Omron_B3F-10xx -> Button_Switch_THT:SW_PUSH_6mm
- moved SW2 0.06 mm to (179.8, 138.2)
Routing:
- net GND: track 370.5 -> 344.5 mm
- net Net-(JP3-Pad1): track 104.9 -> 111.4 mm
